File: monoCtrl/monoCtrl.kicad_sch (KiCad schematic)
At the start: 15 parts, among them J1 Conn_01x08_Pin, J2 Conn_01x08_Pin, J3 Conn_01x08_Pin, J4 Conn_01x08_Pin, J5 Conn_01x08_Pin, J6 Jack-DC

Commit message: finished v0.1
ready to etch
Parts:
- removed J1, J2, J3, J4, J5: Conn_01x08_Pin, uC:1x08_BoardEdge, symbol Connector:Conn_01x08_Pin
- added J1, J2: Conn_01x06_Pin, uC:1x06_BoardEdge, symbol Connector:Conn_01x06_Pin
- added J10, J11, J12, J7, J8, J9: Conn_01x01_Pin, uC:air jump, symbol Connector:Conn_01x01_Pin
- added J3, J4, J5: Conn_01x05_Pin, uC:1x05_BoardEdge, symbol Connector:Conn_01x05_Pin
Connections:
- net +5V: now also J3.5 (Pin_5), J4.5 (Pin_5), J5.5 (Pin_5)
- net GND: now also J10.1 (Pin_1), J11.1 (Pin_1), J12.1 (Pin_1), J3.1 (Pin_1), J3.3 (Pin_3), J4.1 (Pin_1), J4.3 (Pin_3), J5.1 (Pin_1), J5.3 (Pin_3), J7.1 (Pin_1), J8.1 (Pin_1), J9.1 (Pin_1)
- net GratingDetect: now also U1.9 (D9), J5.4 (Pin_4); no longer U1.11 (SDC/D2)
- net GratingDetectLED: now also J5.2 (Pin_2)
- net StallDetect: now also U1.10 (SCL/D3), J3.4 (Pin_4); no longer U1.13 (RX/D0)
- net StallDetectLED: now also J3.2 (Pin_2)
- net ZeroDetect: now also U1.11 (SDC/D2), J4.4 (Pin_4); no longer U1.12 (TX/D1)
- net ZeroDetectLED: now also J4.2 (Pin_2)
- net at A1.3 (A2): now also J1.6 (Pin_6)
- net at A1.4 (A1): now also J1.4 (Pin_4)
- net at A1.5 (B1): now also J1.3 (Pin_3)
- net at A1.6 (B2): now also J1.1 (Pin_1)
- net at A2.6 (B2): now also J2.1 (Pin_1)
- net at A2.5 (B1): now also J2.3 (Pin_3)
- net at A2.4 (A1): now also J2.4 (Pin_4)
- net at A2.3 (A2): now also J2.6 (Pin_6)
