File: DDRN_Hardware/DDRN_Hardware.kicad_sch (KiCad schematic)
At the start: 16 parts, among them J1 SWD, J2 Conn_Coaxial, J3 USB_Comms, SW1 SW_Push, U1 LoRa-E5, U2 MX25R3235FM1xx0, U3 BME280, U4 BMA400

Commit message: pcb design work
Parts:
- removed U2: MX25R3235FM1xx0, Package_SO:SOP-8_3.9x4.9mm_P1.27mm, symbol Memory_Flash:MX25R3235FM1xx0
- removed U3: BME280, Package_LGA:Bosch_LGA-8_2.5x2.5mm_P0.65mm_ClockwisePinNumbering, symbol Sensor:BME280
- removed U4: BMA400, BMA400:XDCR_BMA400, symbol BMA400:BMA400
- added C10, C9: 0.01u, Capacitor_SMD:C_0805_2012Metric_Pad1.18x1.45mm_HandSolder, symbol Device:C_Small
- added C11, C14: 100n, Capacitor_SMD:C_0805_2012Metric_Pad1.18x1.45mm_HandSolder, symbol Device:C_Small
- added C12, C13: 10u, Capacitor_SMD:C_0805_2012Metric_Pad1.18x1.45mm_HandSolder, symbol Device:C_Small
- added C4, C5, C6, C8: 1u, Capacitor_SMD:C_0805_2012Metric_Pad1.18x1.45mm_HandSolder, symbol Device:C_Small
- added C7: 4.7u, Capacitor_SMD:C_0805_2012Metric_Pad1.18x1.45mm_HandSolder, symbol Device:C_Small
- added D2: CDBW46-G, Diode_SMD:D_SOD-123, symbol Device:D_Schottky
- added J4: Conn_01x04_Pin, Library:SLW4S-1C7LF, symbol Connector:Conn_01x04_Pin
- added J5: Conn_01x06_Pin, Library:SLW6S-1C7LF, symbol Connector:Conn_01x06_Pin
- added J6: Conn_01x02_Pin, Library:JST-PH-RH-SM, symbol Connector:Conn_01x02_Pin
- added L1: 150uH, Library:SRN4026, symbol Device:L_Iron
- added Q1, Q2: BSS119, Package_TO_SOT_SMD:SOT-23, symbol Transistor_FET:BSS138
- added R10, R17, R5, R6, R7, R8, R9: 10k, Resistor_SMD:R_0805_2012Metric_Pad1.20x1.40mm_HandSolder, symbol Device:R_Small_US
- added R11: 100, Resistor_SMD:R_0805_2012Metric_Pad1.20x1.40mm_HandSolder, symbol Device:R_Small_US
- added R12: 1k, Resistor_SMD:R_0805_2012Metric_Pad1.20x1.40mm_HandSolder, symbol Device:R_Small_US
- added R13: 4.02k, Resistor_SMD:R_0805_2012Metric_Pad1.20x1.40mm_HandSolder, symbol Device:R_Small_US
- added R14: 2.0k, Resistor_SMD:R_0805_2012Metric_Pad1.20x1.40mm_HandSolder, symbol Device:R_Small_US
- added R15: 205k, Resistor_SMD:R_0805_2012Metric_Pad1.20x1.40mm_HandSolder, symbol Device:R_Small_US
- added R16: 32.4k, Resistor_SMD:R_0805_2012Metric_Pad1.20x1.40mm_HandSolder, symbol Device:R_Small_US
- added U2: MAX1932, Package_DFN_QFN:DFN-12-1EP_4x4mm_P0.65mm_EP2.64x3.54mm, symbol MAX1932:MAX1932
- added U3: BMP390L, BMP390L:XDCR_BMP390L, symbol BMP390L:BMP390L
- added U4: W25Q32JVSS, Package_SO:SOIC-8_5.23x5.23mm_P1.27mm, symbol Memory_Flash:W25Q32JVSS
- added U5: ADXL343, Package_LGA:LGA-14_3x5mm_P0.8mm_LayoutBorder1x6y, symbol Sensor_Motion:ADXL343
- added U6: AP2112K-3.3, Package_TO_SOT_SMD:SOT-23-5, symbol Regulator_Linear:AP2112K-3.3
Connections:
- net 3v3: now also C13.1, C14.1, C4.1, C5.1, C6.1, C7.1, J5.1 (Pin_1), R12.2, R6.2, R7.2, R8.2, U3.1 (VDDIO), U3.10 (VDD), U4.8 (VCC), U5.1 (Vdd_I/O), U5.6 (Vs), U6.5 (VOUT); no longer J3.1 (VCC)
- net Anneal_Enable: now also J4.4 (Pin_4)
- net Battery_Monitor: now also R11.1
- net Bias_CS: now also U2.12 (CS)
- net GND: now also C10.2, C11.2, C12.2, C13.2, C14.2, C4.2, C5.2, C6.2, C7.2, C8.2, C9.2, J4.2 (Pin_2), J5.4 (Pin_4), J6.2 (Pin_2), Q1.2 (S), Q2.2 (S), R17.2, R5.2, U2.13 (PAN), U2.9 (GND), U3.3 (VSS/GND), U3.8 (VSS/GND), U3.9 (VSS/GND), U4.4 (GND), U5.2 (GND), U5.4 (GND), U5.5 (GND), U6.2 (GND)
- net MISO: now also U4.2 (DO(IO1))
- net MOSI: now also U2.2 (MOSI), U4.5 (DI(IO0))
- net Memory_CS: now also U4.1 (~{CS})
- net RST: now also R12.1
- net SCK: now also U2.1 (SCLK), U4.6 (CLK)
- net SCL: now also U3.2 (SCK/SCL), U5.14 (SCL/SCLK)
- net SDA: now also U3.4 (SDI/SDO/SDA), U5.13 (SDA/SDI/SDIO)
- net SiPM_Signal: now also J5.5 (Pin_5)
- net SiPM_Temp: now also J5.2 (Pin_2)
- net Stim_Enable: now also J4.3 (Pin_3)
- net ACCEL_INT: now reaches U1.13 (PC0)
- net ACCEL_INT: now also U5.8 (INT1)
- net Battery_Monitor_Enable: now reaches U1.20 (PB10)
- net Battery_Monitor_Enable: now also Q1.1 (G)
- new net: R6.1, U5.7 (~{CS})
- new net: R10.1, R11.2, R9.2
- new net: Q2.1 (G), U2.10 (GATE)
- new net: D2.2 (A), L1.2, Q2.3 (D)
- new net: R16.1, U2.6 (DACOUT)
- new net: R15.2, R16.2, R17.1, U2.7 (FB)
- new net: C9.1, D2.1 (K), R14.1, U2.4 (CS+)
- new net: R13.2, U2.8 (COMP)
- new net: Q1.3 (D), R10.2
- new net: R5.1, U5.12 (SDO/ADDR)
- new net: C8.1, R13.1
- new net: R7.1, U3.5 (SDO/DNC/SA0)
- new net: R8.1, U3.6 (~{CS})
- new net 5v: C11.1, C12.1, J3.1 (VCC), U6.1 (VIN), U6.3 (EN)
- new net SiPM_Bias: C10.1, J5.3 (Pin_3), R14.2, R15.1, U2.5 (CS-)
- new net V_BAT: J4.1 (Pin_1), J5.6 (Pin_6), J6.1 (Pin_1), L1.1, R9.1, U2.11 (VIN)
- no-connect marks 10 -> 7
Other:
- moved on the sheet: R3, R4, SW1
