File: DDRN_Hardware/DDRN_Hardware.kicad_sch (KiCad schematic)
At the start: 36 parts, among them J1 SWD, J2 Conn_01x02_Pin, J3 Conn_01x04_Pin, J4 Conn_01x06_Pin, J7 Conn_02x12_Counter_Clockwise, Q1 BSS119, Q2 BSS119, U1 MAX1932, U2 LoRa-E5, U3 BMP390L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

Commit message: kicad correction
Changed lines of the file:
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@@
     )
   )
-  (sheet (at 83.82 17.78) (size 43.18 34.29) (fields_autoplaced)
+  (sheet (at 82.55 26.67) (size 43.18 34.29) (fields_autoplaced)
     (stroke (width 0.1524) (type solid))
     (fill (color 0 0 0 0.0000))
-    (property "Sheetname" "E5_mini_dev_items" (at 83.82 17.0684 0)
+    (property "Sheetname" "E5_mini_dev_items" (at 82.55 25.9584 0)
       (effects (font (size 1.27 1.27)) (justify left bottom))
     )
-    (property "Sheetfile" "E5_mini_dev_items.kicad_sch" (at 83.82 52.6546 0)
+    (property "Sheetfile" "E5_mini_dev_items.kicad_sch" (at 82.55 61.5446 0)
       (effects (font (size 1.27 1.27)) (justify left top))
     )
