File: DDRN_Hardware/DDRN_Hardware.kicad_pcb (KiCad board)
At the start: 2 copper layers, 16 parts, among them J1 SWD, J2 Conn_Coaxial, J3 USB_Comms, SW1 SW_Push, U1 LoRa-E5, U2 MX25R3235FM1xx0, U3 BME280, U4 BMA400

Commit message: pcb design work
Parts:
- added C10: 0.01u, Capacitor_SMD:C_0805_2012Metric_Pad1.18x1.45mm_HandSolder, F.Cu at (112.8, 64.6)
- added C11: 100n, Capacitor_SMD:C_0805_2012Metric_Pad1.18x1.45mm_HandSolder, F.Cu at (106.9, 30.1)
- added C12: 10u, Capacitor_SMD:C_0805_2012Metric_Pad1.18x1.45mm_HandSolder, F.Cu at (106.9, 33.1)
- added C13: 10u, Capacitor_SMD:C_0805_2012Metric_Pad1.18x1.45mm_HandSolder, F.Cu at (106.9, 36.1)
- added C14: 100n, Capacitor_SMD:C_0805_2012Metric_Pad1.18x1.45mm_HandSolder, F.Cu at (106.9, 39.1)
- added C4: 1u, Capacitor_SMD:C_0805_2012Metric_Pad1.18x1.45mm_HandSolder, F.Cu at (108.0, 61.6)
- added C5: 1u, Capacitor_SMD:C_0805_2012Metric_Pad1.18x1.45mm_HandSolder, F.Cu at (108.0, 64.6)
- added C6: 1u, Capacitor_SMD:C_0805_2012Metric_Pad1.18x1.45mm_HandSolder, F.Cu at (112.8, 52.5)
- added C7: 4.7u, Capacitor_SMD:C_0805_2012Metric_Pad1.18x1.45mm_HandSolder, F.Cu at (112.8, 55.5)
- added C8: 1u, Capacitor_SMD:C_0805_2012Metric_Pad1.18x1.45mm_HandSolder, F.Cu at (112.8, 58.5)
- added C9: 0.01u, Capacitor_SMD:C_0805_2012Metric_Pad1.18x1.45mm_HandSolder, F.Cu at (112.8, 61.6)
- added D2: CDBW46-G, Diode_SMD:D_SOD-123, F.Cu at (112.2, 68.0)
- added J4: Conn_01x04_Pin, Library:SLW4S-1C7LF, F.Cu at (122.8, 81.5)
- added J5: Conn_01x06_Pin, Library:SLW6S-1C7LF, F.Cu at (118.3, 77.0)
- added J6: Conn_01x02_Pin, Library:JST-PH-RH-SM, F.Cu at (63.3, 51.6)
- added L1: 150uH, Library:SRN4026, F.Cu at (116.8, 81.9)
- added Q1: BSS119, Package_TO_SOT_SMD:SOT-23, F.Cu at (86.3, 70.9)
- added Q2: BSS119, Package_TO_SOT_SMD:SOT-23, F.Cu at (86.3, 75.4)
- added R10: 10k, Resistor_SMD:R_0805_2012Metric_Pad1.20x1.40mm_HandSolder, F.Cu at (82.9, 61.3)
- added R11: 100, Resistor_SMD:R_0805_2012Metric_Pad1.20x1.40mm_HandSolder, F.Cu at (82.9, 64.3)
- added R12: 1k, Resistor_SMD:R_0805_2012Metric_Pad1.20x1.40mm_HandSolder, F.Cu at (82.9, 67.2)
- added R13: 4.02k, Resistor_SMD:R_0805_2012Metric_Pad1.20x1.40mm_HandSolder, F.Cu at (87.7, 52.5)
- added R14: 2.0k, Resistor_SMD:R_0805_2012Metric_Pad1.20x1.40mm_HandSolder, F.Cu at (87.7, 55.4)
- added R15: 205k, Resistor_SMD:R_0805_2012Metric_Pad1.20x1.40mm_HandSolder, F.Cu at (87.7, 58.4)
- added R16: 32.4k, Resistor_SMD:R_0805_2012Metric_Pad1.20x1.40mm_HandSolder, F.Cu at (87.7, 61.3)
- added R17: 10k, Resistor_SMD:R_0805_2012Metric_Pad1.20x1.40mm_HandSolder, F.Cu at (87.7, 64.3)
- added R5: 10k, Resistor_SMD:R_0805_2012Metric_Pad1.20x1.40mm_HandSolder, F.Cu at (78.2, 64.3)
- added R6: 10k, Resistor_SMD:R_0805_2012Metric_Pad1.20x1.40mm_HandSolder, F.Cu at (78.2, 67.2)
- added R7: 10k, Resistor_SMD:R_0805_2012Metric_Pad1.20x1.40mm_HandSolder, F.Cu at (82.9, 52.5)
- added R8: 10k, Resistor_SMD:R_0805_2012Metric_Pad1.20x1.40mm_HandSolder, F.Cu at (82.9, 55.4)
- added R9: 10k, Resistor_SMD:R_0805_2012Metric_Pad1.20x1.40mm_HandSolder, F.Cu at (82.9, 58.4)
- added U5: ADXL343, Package_LGA:LGA-14_3x5mm_P0.8mm_LayoutBorder1x6y, F.Cu at (78.1, 82.1)
- added U6: AP2112K-3.3, Package_TO_SOT_SMD:SOT-23-5, F.Cu at (111.9, 30.8)
- U2: value MX25R3235FM1xx0 -> MAX1932; footprint Package_SO:SOP-8_3.9x4.9mm_P1.27mm -> Package_DFN_QFN:DFN-12-1EP_4x4mm_P0.65mm_EP2.64x3.54mm
- U3: value BME280 -> BMP390L; footprint Package_LGA:Bosch_LGA-8_2.5x2.5mm_P0.65mm_ClockwisePinNumbering -> BMP390L:XDCR_BMP390L
- U4: value BMA400 -> W25Q32JVSS; footprint BMA400:XDCR_BMA400 -> Package_SO:SOIC-8_5.23x5.23mm_P1.27mm
- moved U3 41.3 mm to (88.0, 81.1)
- moved U2 39.8 mm to (83.3, 81.7)
- moved R3 34.1 mm to (78.2, 58.4)
- moved R4 34.1 mm to (78.2, 61.3)
- moved J2 31.4 mm to (94.3, 72.4)
- moved D1 28.1 mm to (111.7, 71.2)
- moved SW1 25.8 mm to (95.6, 82.8)
- moved U4 22.9 mm to (106.3, 81.9)
- moved C1 20.2 mm to (108.0, 52.5)
- moved C2 20.2 mm to (108.0, 55.5)
- moved C3 20.2 mm to (108.0, 58.5)
- moved R1 16.5 mm to (78.2, 52.5)
- moved R2 16.5 mm to (78.2, 55.4)
- moved J3 14.4 mm to (79.8, 76.3)
- moved J1 12.3 mm to (79.8, 71.2)
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Connections:
- J3 pad 1: /3v3 -> /5v
- U1 pad 13: unconnected-(U1-PC0-Pad13) -> /ACCEL_INT
- U1 pad 20: unconnected-(U1-PB10-Pad20) -> /Battery_Monitor_Enable
- U2 pad 1: /Memory_CS -> /SCK
- U2 pad 2: /MISO -> /MOSI
- U2 pad 4: GND -> Net-(D2-K)
- U2 pad 5: /MOSI -> /SiPM_Bias
- U2 pad 6: /SCK -> Net-(U2-DACOUT)
- U2 pad 7: unconnected-(U2-~{RESET}/SIO3-Pad7) -> Net-(U2-FB)
- U2 pad 8: /3v3 -> Net-(U2-COMP)
- U3 pad 1: GND -> /3v3
- U3 pad 2: /3v3 -> /SCL
- U3 pad 3: /SDA -> GND
- U3 pad 4: /SCL -> /SDA
- U3 pad 5: /3v3 -> Net-(U3-SDO/DNC/SA0)
- U3 pad 6: /3v3 -> Net-(U3-~{CS})
- U3 pad 7: GND -> unconnected-(U3-INT/DNC-Pad7)
- U3 pad 8: /3v3 -> GND
- U4 pad 1: unconnected-(U4-SDO-Pad1) -> /Memory_CS
- U4 pad 2: /SDA -> /MISO
- U4 pad 3: /3v3 -> unconnected-(U4-IO2-Pad3)
- U4 pad 4: (no net) -> GND
- U4 pad 5: unconnected-(U4-INT1-Pad5) -> /MOSI
- U4 pad 6: unconnected-(U4-INT2-Pad6) -> /SCK
- U4 pad 7: /3v3 -> unconnected-(U4-IO3-Pad7)
- U4 pad 8: GND -> /3v3

Commit message: pcb v1 work
Parts:
- removed C10, C9: 0.01u, Capacitor_SMD:C_0805_2012Metric_Pad1.18x1.45mm_HandSolder
- removed C11, C14: 100n, Capacitor_SMD:C_0805_2012Metric_Pad1.18x1.45mm_HandSolder
- removed C12, C13: 10u, Capacitor_SMD:C_0805_2012Metric_Pad1.18x1.45mm_HandSolder
- removed C2: DNP, Capacitor_SMD:C_0805_2012Metric_Pad1.18x1.45mm_HandSolder
- removed D2: CDBW46-G, Diode_SMD:D_SOD-123
- removed J5: Conn_01x06_Pin, Library:SLW6S-1C7LF
- removed J6: Conn_01x02_Pin, Library:JST-PH-RH-SM
- removed R15: 205k, Resistor_SMD:R_0805_2012Metric_Pad1.20x1.40mm_HandSolder
- removed R16: 32.4k, Resistor_SMD:R_0805_2012Metric_Pad1.20x1.40mm_HandSolder
- removed R17: 10k, Resistor_SMD:R_0805_2012Metric_Pad1.20x1.40mm_HandSolder
- removed SW1: SW_Push, Button_Switch_SMD:SW_SPST_B3S-1000
- removed U2: MAX1932, Package_DFN_QFN:DFN-12-1EP_4x4mm_P0.65mm_EP2.64x3.54mm
- removed U6: AP2112K-3.3, Package_TO_SOT_SMD:SOT-23-5
- added J7: Conn_02x12_Counter_Clockwise, Library:E5-mini-dev, B.Cu at (121.9, 77.5)
- C3: value DNP -> 1u
- C4, C5: value 1u -> 0.01u
- C7: value 4.7u -> 1u
- D1: value LED -> CDBW46-G; footprint LED_SMD:LED_0805_2012Metric_Pad1.15x1.40mm_HandSolder -> Diode_SMD:D_SOD-123
- J2: value Conn_Coaxial -> Conn_01x02_Pin; footprint Connector_Coaxial:SMA_Amphenol_132289_EdgeMount -> Library:JST-PH-RH-SM
- J3: value USB_Comms -> Conn_01x04_Pin; footprint Connector:Tag-Connect_TC2030-IDC-NL_2x03_P1.27mm_Vertical -> Library:SLW4S-1C7LF; moved to B.Cu
- J4: value Conn_01x04_Pin -> Conn_01x06_Pin; footprint Library:SLW4S-1C7LF -> Library:SLW6S-1C7LF; moved to B.Cu
- R1: value 1k -> 4.02k
- R10: value 10k -> 4.7k
- R11: value 100 -> 4.7k
- R12: value 1k -> 10k
- R13: value 4.02k -> 10k
- R14: value 2.0k -> 100
- R2: value 0R -> 32.4k
- R3: value 4.7k -> 2.0k
- R4: value 4.7k -> 205k
- U1: value LoRa-E5 -> MAX1932; footprint LoRa-E5:LoRa-E5 -> Package_DFN_QFN:DFN-12-1EP_4x4mm_P0.65mm_EP2.64x3.54mm
- U4: value W25Q32JVSS -> ADXL343; footprint Package_SO:SOIC-8_5.23x5.23mm_P1.27mm -> Package_LGA:LGA-14_3x5mm_P0.8mm_LayoutBorder1x6y
- U5: value ADXL343 -> W25Q32JVSS; footprint Package_LGA:LGA-14_3x5mm_P0.8mm_LayoutBorder1x6y -> Package_SO:SOIC-8_5.23x5.23mm_P1.27mm
- moved R4 98.8 mm to (176.8, 55.9)
- moved R3 98.6 mm to (176.5, 52.1)
- moved R5 96.5 mm to (174.6, 61.0)
- moved R2 92.7 mm to (170.4, 46.4)
- moved R1 87.9 mm to (165.4, 41.9)
- moved Q1 86.8 mm to (170.8, 51.4)
- moved D1 67.6 mm to (174.6, 46.4), turned to 90 degrees
- moved U1 63.6 mm to (160.0, 44.9)
- moved C5 63.1 mm to (170.6, 56.5)
- moved J3 59.8 mm to (138.7, 86.9), turned to 90 degrees
- moved C4 58.4 mm to (166.0, 54.6)
- moved C3 57.9 mm to (165.3, 50.2)
- moved C1 57.7 mm to (165.3, 46.4)
- moved R9 54.5 mm to (136.2, 47.0)
- moved R8 54.1 mm to (136.8, 50.2)
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Connections:
- C3 pad 1: Net-(J2-In) -> Net-(C3-Pad1)
- C4 pad 1: /3v3 -> Net-(D1-K)
- C5 pad 1: /3v3 -> /SiPM_Bias
- C8 pad 1: Net-(C8-Pad1) -> /3v3
- D1 pad 1: /Status_LED -> Net-(D1-K)
- J2 pad 1: Net-(J2-In) -> /V_BAT
- J3 pad 1: /5v -> /V_BAT
- J3 pad 2: unconnected-(J3-SWDIO-Pad2) -> GND
- J3 pad 3: /USB_TX -> /Stim_Enable
- J3 pad 4: /USB_RX -> /Anneal_Enable
- J4 pad 1: /V_BAT -> /3v3
- J4 pad 2: GND -> /SiPM_Temp
- J4 pad 3: /Stim_Enable -> /SiPM_Bias
- J4 pad 4: /Anneal_Enable -> GND
- L1 pad 2: Net-(D2-A) -> Net-(D1-A)
- Q1 pad 1: /Battery_Monitor_Enable -> Net-(Q1-G)
- Q1 pad 3: Net-(Q1-D) -> Net-(D1-A)
- Q2 pad 1: Net-(Q2-G) -> /Battery_Monitor_Enable
- Q2 pad 3: Net-(D2-A) -> Net-(Q2-D)
- R1 pad 1: Net-(D1-A) -> Net-(C3-Pad1)
- R1 pad 2: /3v3 -> Net-(U1-COMP)
- R10 pad 1: Net-(R10-Pad1) -> /SCL
- R10 pad 2: Net-(Q1-D) -> /3v3
- R11 pad 1: /Battery_Monitor -> /SDA
- R11 pad 2: Net-(R10-Pad1) -> /3v3
- R12 pad 1: /RST -> /V_BAT
- R12 pad 2: /3v3 -> Net-(R12-Pad2)
- R13 pad 1: Net-(C8-Pad1) -> Net-(R12-Pad2)
- R13 pad 2: Net-(U2-COMP) -> Net-(Q2-D)
- R14 pad 1: Net-(D2-K) -> /Battery_Monitor
- R14 pad 2: /SiPM_Bias -> Net-(R12-Pad2)
- R2 pad 1: Net-(J2-In) -> Net-(U1-DACOUT)
- R2 pad 2: /ANT -> Net-(U1-FB)
- R3 pad 1: /SCL -> Net-(D1-K)
- R3 pad 2: /3v3 -> /SiPM_Bias
- R4 pad 1: /SDA -> /SiPM_Bias
- R4 pad 2: /3v3 -> Net-(U1-FB)
- R5 pad 1: Net-(U5-SDO/ADDR) -> Net-(U1-FB)
- R6 pad 1: Net-(U5-~{CS}) -> Net-(U3-~{CS})
- R8 pad 1: Net-(U3-~{CS}) -> Net-(U4-SDO/ADDR)
- R8 pad 2: /3v3 -> GND
- R9 pad 1: /V_BAT -> Net-(U4-~{CS})
- R9 pad 2: Net-(R10-Pad1) -> /3v3
- U1 pad 1: /3v3 -> /SCK
- U1 pad 10: /USB_TX -> Net-(Q1-G)
- U1 pad 11: /Status_LED -> /V_BAT
- U1 pad 12: /MOSI -> /Bias_CS
- U1 pad 13: /ACCEL_INT -> GND
- U1 pad 2: GND -> /MOSI
- U1 pad 3: /SWDIO -> unconnected-(U1-CL-Pad3)
- U1 pad 4: /SWCLK -> Net-(D1-K)
- U1 pad 5: /SCL -> /SiPM_Bias
- U1 pad 6: /SDA -> Net-(U1-DACOUT)
- U1 pad 7: /SiPM_Signal -> Net-(U1-FB)
- U1 pad 8: /SiPM_Temp -> Net-(U1-COMP)
- U1 pad 9: /USB_RX -> GND
- U4 pad 1: /Memory_CS -> /3v3
- U4 pad 2: /MISO -> GND
- U4 pad 5: /MOSI -> GND
- U4 pad 6: /SCK -> /3v3
- U4 pad 7: unconnected-(U4-IO3-Pad7) -> Net-(U4-~{CS})
- U4 pad 8: /3v3 -> /ACCEL_INT
- U5 pad 1: /3v3 -> /Memory_CS
- U5 pad 2: GND -> /MISO
- U5 pad 5: GND -> /MOSI
- U5 pad 6: /3v3 -> /SCK
- U5 pad 7: Net-(U5-~{CS}) -> unconnected-(U5-IO3-Pad7)
- U5 pad 8: /ACCEL_INT -> /3v3
Routing:
- net /3v3: track 0.00 -> 53.7 mm
- net /MOSI: track 0.00 -> 35.2 mm
- net /SCK: track 0.00 -> 20.9 mm
- net /RST: track 0.00 -> 13.7 mm
- net /Memory_CS: track 0.00 -> 7.61 mm
- net /SWDIO: track 0.00 -> 7.51 mm
- net /MISO: track 0.00 -> 7.09 mm
- net /SWCLK: track 0.00 -> 6.98 mm
- net GND: track 0.00 -> 6.74 mm
- net Net-(U3-~{CS}): track 0.00 -> 2.95 mm
- net Net-(U3-SDO/DNC/SA0): track 0.00 -> 2.79 mm
- net /SDA: track 0.00 -> 2.44 mm
- net /SCL: track 0.00 -> 2.44 mm
- added copper zone on F.Cu, net GND
Other:
- board outline added: 52.1 x 49.5 mm

Commit message: kicad correction
Parts:
- moved C1 8.41 mm to (167.9, 54.4)
- moved C3 8.41 mm to (167.9, 58.2)
- moved C4 8.41 mm to (168.6, 62.6)
- moved D1 8.41 mm to (177.2, 54.4)
- moved L1 8.41 mm to (162.6, 60.1)
- moved R1 8.41 mm to (168.0, 49.9)
- moved R2 8.41 mm to (173.0, 54.4)
- moved R3 8.41 mm to (179.1, 60.1)
- moved R5 8.41 mm to (177.2, 69.0)
- moved U1 8.41 mm to (162.6, 52.9)
- moved C5 8.41 mm to (173.2, 64.5)
- moved Q1 8.41 mm to (173.4, 59.4)
- moved R4 8.41 mm to (179.4, 63.9)
Changed lines of the file:
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@@
   (net 47 "/5v")
   (footprint "Diode_SMD:D_SOD-123" (layer "F.Cu")
-    (at 174.625 46.355 90)
+    (at 177.215 54.36 90)
     (descr "SOD-123")
     (tags "SOD-123")
@@
   )
   (footprint "Capacitor_SMD:C_0805_2012Metric_Pad1.18x1.45mm_HandSolder" (layer "F.Cu")
-    (at 170.605 56.515)
+    (at 173.195 64.52)
     (descr "Capacitor SMD 0805 (2012 Metric), square (rectangular) end terminal, IPC_7351 nominal with elongated pad for handsoldering. (Body size source: IPC-SM-782 page 76, https://www.pcb-3d.com/wordpress/wp-content/uploads/ipc-sm-782a_amendment_1_and_2.pdf, https://docs.google.com/spreadsheets/d/1BsfQQcO9C6DZCsRaXUlFlo91Tg2WpOkGARC1WS5S8t0/edit?usp=sharing), generated with kicad-footprint-generator")
     (tags "capacitor handsolder")
@@
   )
   (footprint "Capacitor_SMD:C_0805_2012Metric_Pad1.18x1.45mm_HandSolder" (layer "F.Cu")
-    (at 165.3325 50.165)
+    (at 167.9225 58.17)
     (descr "Capacitor SMD 0805 (2012 Metric), square (rectangular) end terminal, IPC_7351 nominal with elongated pad for handsoldering. (Body size source: IPC-SM-782 page 76, https://www.pcb-3d.com/wordpress/wp-content/uploads/ipc-sm-782a_amendment_1_and_2.pdf, https://docs.google.com/spreadsheets/d/1BsfQQcO9C6DZCsRaXUlFlo91Tg2WpOkGARC1WS5S8t0/edit?usp=sharing), generated with kicad-footprint-generator")
     (tags "capacitor handsolder")
@@
   )
   (footprint "Capacitor_SMD:C_0805_2012Metric_Pad1.18x1.45mm_HandSolder" (layer "F.Cu")
-    (at 165.9675 54.61)
+    (at 168.5575 62.615)
     (descr "Capacitor SMD 0805 (2012 Metric), square (rectangular) end terminal, IPC_7351 nominal with elongated pad for handsoldering. (Body size source: IPC-SM-782 page 76, https://www.pcb-3d.com/wordpress/wp-content/uploads/ipc-sm-782a_amendment_1_and_2.pdf, https://docs.google.com/spreadsheets/d/1BsfQQcO9C6DZCsRaXUlFlo91Tg2WpOkGARC1WS5S8t0/edit?usp=sharing), generated with kicad-footprint-generator")
     (tags "capacitor handsolder")
@@
   )
   (footprint "Resistor_SMD:R_0805_2012Metric_Pad1.20x1.40mm_HandSolder" (layer "F.Cu")
-    (at 174.625 60.96)
+    (at 177.215 68.965)
     (descr "Resistor SMD 0805 (2012 Metric), square (rectangular) end terminal, IPC_7351 nominal with elongated pad for handsoldering. (Body size source: IPC-SM-782 page 72, https://www.pcb-3d.com/wordpress/wp-content/uploads/ipc-sm-782a_amendment_1_and_2.pdf), generated with kicad-footprint-generator")
     (tags "resistor handsolder")
@@
   )
   (footprint "Library:SRN4026" (layer "F.Cu")
-    (at 160.02 52.07)
+    (at 162.61 60.075)
     (property "Sheetfile" "DDRN_Hardware.kicad_sch")
     (property "Sheetname" "")
@@
   )
   (footprint "Package_DFN_QFN:DFN-12-1EP_4x4mm_P0.65mm_EP2.64x3.54mm" (layer "F.Cu")
-    (at 159.995 44.8925)
+    (at 162.585 52.8975)
     (descr "DFN12, 4x4, 0.65P; CASE 506CE (see ON Semiconductor 506CE.PDF)")
     (tags "DFN 0.65")
@@
   )
   (footprint "Resistor_SMD:R_0805_2012Metric_Pad1.20x1.40mm_HandSolder" (layer "F.Cu")
-    (at 165.37 41.91)
+    (at 167.96 49.915)
     (descr "Resistor SMD 0805 (2012 Metric), square (rectangular) end terminal, IPC_7351 nominal with elongated pad for handsoldering. (Body size source: IPC-SM-782 page 72, https://www.pcb-3d.com/wordpress/wp-content/uploads/ipc-sm-782a_amendment_1_and_2.pdf), generated with kicad-footprint-generator")
     (tags "resistor handsolder")
@@
   )
   (footprint "Resistor_SMD:R_0805_2012Metric_Pad1.20x1.40mm_HandSolder" (layer "F.Cu")
-    (at 176.53 52.07)
+    (at 179.12 60.075)
     (descr "Resistor SMD 0805 (2012 Metric), square (rectangular) end terminal, IPC_7351 nominal with elongated pad for handsoldering. (Body size source: IPC-SM-782 page 72, https://www.pcb-3d.com/wordpress/wp-content/uploads/ipc-sm-782a_amendment_1_and_2.pdf), generated with kicad-footprint-generator")
     (tags "resistor handsolder")
@@
   )
   (footprint "Package_TO_SOT_SMD:SOT-23" (layer "F.Cu")
-    (at 170.815 51.435)
+    (at 173.405 59.44)
     (descr "SOT, 3 Pin (https://www.jedec.org/system/files/docs/to-236h.pdf variant AB), generated with kicad-footprint-generator ipc_gullwing_generator.py")
     (tags "SOT TO_SOT_SMD")
@@
   )
   (footprint "Capacitor_SMD:C_0805_2012Metric_Pad1.18x1.45mm_HandSolder" (layer "F.Cu")
-    (at 165.3325 46.355)
+    (at 167.9225 54.36)
     (descr "Capacitor SMD 0805 (2012 Metric), square (rectangular) end terminal, IPC_7351 nominal with elongated pad for handsoldering. (Body size source: IPC-SM-782 page 76, https://www.pcb-3d.com/wordpress/wp-content/uploads/ipc-sm-782a_amendment_1_and_2.pdf, https://docs.google.com/spreadsheets/d/1BsfQQcO9C6DZCsRaXUlFlo91Tg2WpOkGARC1WS5S8t0/edit?usp=sharing), generated with kicad-footprint-generator")
     (tags "capacitor handsolder")
@@
   )
   (footprint "Resistor_SMD:R_0805_2012Metric_Pad1.20x1.40mm_HandSolder" (layer "F.Cu")
-    (at 170.45 46.355)
+    (at 173.04 54.36)
     (descr "Resistor SMD 0805 (2012 Metric), square (rectangular) end terminal, IPC_7351 nominal with elongated pad for handsoldering. (Body size source: IPC-SM-782 page 72, https://www.pcb-3d.com/wordpress/wp-content/uploads/ipc-sm-782a_amendment_1_and_2.pdf), generated with kicad-footprint-generator")
     (tags "resistor handsolder")
@@
   )
   (footprint "Resistor_SMD:R_0805_2012Metric_Pad1.20x1.40mm_HandSolder" (layer "F.Cu")
-    (at 176.8 55.88)
+    (at 179.39 63.885)
     (descr "Resistor SMD 0805 (2012 Metric), square (rectangular) end terminal, IPC_7351 nominal with elongated pad for handsoldering. (Body size source: IPC-SM-782 page 72, https://www.pcb-3d.com/wordpress/wp-content/uploads/ipc-sm-782a_amendment_1_and_2.pdf), generated with kicad-footprint-generator")
     (tags "resistor handsolder")
