File: DDRN_Hardware/v0.1/DDRN_Hardware.kicad_sch (KiCad schematic)
At the start: 45 parts, among them J2 Conn_Coaxial, J3 Conn_01x02_Pin, J4 Conn_01x04_Pin, J5 Conn_01x06_Pin, J8 Conn_02x05_Top_Bottom, Q1 BSS119, Q2 BSS119, SW1 SW_Push, U1 LoRa-E5, U2 MAX1932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

Commit message: v0.1 pcb complete?
Parts:
- added H1, H2, H3, H4: MountingHole, MountingHole:MountingHole_3.2mm_M3_DIN965, symbol Mechanical:MountingHole
- U5: footprint Library:bmp390_handsolder -> Library:lsm303_handsolder
Connections:
- net Anneal_Enable: now also U1.27 (PA10); no longer U1.23 (PA0)
- net Battery_Monitor_Enable: now also U1.23 (PA0); no longer U1.20 (PB10)
- net Bias_CS: now also U1.20 (PB10); no longer U1.27 (PA10)
- net Memory_CS: now also U1.19 (PA2); no longer U1.25 (PB9)
- net Stim_Enable: now also U1.25 (PB9); no longer U1.19 (PA2)
- net Bias_Enable: no longer names the net of U1.18 (PA3)
Changed lines of the file:
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@@
     (effects (font (size 1.27 1.27)) (justify right bottom))
   )
-  (label "Stim_Enable" (at 139.7 100.33 0) (fields_autoplaced)
+  (label "Stim_Enable" (at 121.92 85.09 90) (fields_autoplaced)
     (effects (font (size 1.27 1.27)) (justify left bottom))
   )
@@
     (effects (font (size 1.27 1.27)) (justify right bottom))
   )
-  (label "Bias_Enable" (at 139.7 102.87 0) (fields_autoplaced)
-    (effects (font (size 1.27 1.27)) (justify left bottom))
-  )
   (label "3v3" (at 104.14 95.25 180) (fields_autoplaced)
     (effects (font (size 1.27 1.27)) (justify right bottom))
@@
     (effects (font (size 1.27 1.27)) (justify right bottom))
   )
-  (label "Battery_Monitor_Enable" (at 139.7 97.79 0) (fields_autoplaced)
+  (label "Battery_Monitor_Enable" (at 127 85.09 90) (fields_autoplaced)
     (effects (font (size 1.27 1.27)) (justify left bottom))
   )
@@
     (effects (font (size 1.27 1.27)) (justify left bottom))
   )
-  (label "Memory_CS" (at 121.92 85.09 90) (fields_autoplaced)
+  (label "Memory_CS" (at 139.7 100.33 0) (fields_autoplaced)
     (effects (font (size 1.27 1.27)) (justify left bottom))
   )
@@
     (effects (font (size 1.27 1.27)) (justify left bottom))
   )
-  (label "Anneal_Enable" (at 127 85.09 90) (fields_autoplaced)
+  (label "Anneal_Enable" (at 116.84 85.09 90) (fields_autoplaced)
     (effects (font (size 1.27 1.27)) (justify left bottom))
   )
@@
     (effects (font (size 1.27 1.27)) (justify left bottom))
   )
-  (label "Bias_CS" (at 116.84 85.09 90) (fields_autoplaced)
+  (label "Bias_CS" (at 139.7 97.79 0) (fields_autoplaced)
     (effects (font (size 1.27 1.27)) (justify left bottom))
   )
@@
     )
   )
+  (symbol (lib_id "Mechanical:MountingHole") (at 222.25 80.01 0) (unit 1)
+    (in_bom yes) (on_board yes) (dnp no) (fields_autoplaced)
+    (property "Reference" "H3" (at 224.79 78.74 0)
+      (effects (font (size 1.27 1.27)) (justify left))
+    )
+    (property "Value" "MountingHole" (at 224.79 81.28 0)
+      (effects (font (size 1.27 1.27)) (justify left))
+    )
+    (property "Footprint" "MountingHole:MountingHole_3.2mm_M3_DIN965" (at 222.25 80.01 0)
+      (effects (font (size 1.27 1.27)) hide)
+    )
+    (property "Datasheet" "~" (at 222.25 80.01 0)
+      (effects (font (size 1.27 1.27)) hide)
+    )
+    (instances
+      (project "DDRN_Hardware"
+        (path "/6ac82b7e-9b2f-410f-b4a2-ac71ebf885a9"
+          (reference "H3") (unit 1)
+        )
+      )
+    )
+  )
   (symbol (lib_id "Device:R_Small_US") (at 144.78 158.75 270) (unit 1)
     (in_bom yes) (on_board yes) (dnp no) (fields_autoplaced)
@@
     )
   )
+  (symbol (lib_id "Mechanical:MountingHole") (at 222.25 74.93 0) (unit 1)
+    (in_bom yes) (on_board yes) (dnp no) (fields_autoplaced)
+    (property "Reference" "H2" (at 224.79 73.66 0)
+      (effects (font (size 1.27 1.27)) (justify left))
+    )
+    (property "Value" "MountingHole" (at 224.79 76.2 0)
+      (effects (font (size 1.27 1.27)) (justify left))
+    )
+    (property "Footprint" "MountingHole:MountingHole_3.2mm_M3_DIN965" (at 222.25 74.93 0)
+      (effects (font (size 1.27 1.27)) hide)
+    )
+    (property "Datasheet" "~" (at 222.25 74.93 0)
+      (effects (font (size 1.27 1.27)) hide)
+    )
+    (instances
+      (project "DDRN_Hardware"
+        (path "/6ac82b7e-9b2f-410f-b4a2-ac71ebf885a9"
+          (reference "H2") (unit 1)
+        )
+      )
+    )
+  )
   (symbol (lib_id "Device:R_Small_US") (at 257.81 38.1 0) (unit 1)
     (in_bom yes) (on_board yes) (dnp no) (fields_autoplaced)
@@
     )
   )
+  (symbol (lib_id "Mechanical:MountingHole") (at 222.25 85.09 0) (unit 1)
+    (in_bom yes) (on_board yes) (dnp no) (fields_autoplaced)
+    (property "Reference" "H4" (at 224.79 83.82 0)
+      (effects (font (size 1.27 1.27)) (justify left))
+    )
+    (property "Value" "MountingHole" (at 224.79 86.36 0)
+      (effects (font (size 1.27 1.27)) (justify left))
+    )
+    (property "Footprint" "MountingHole:MountingHole_3.2mm_M3_DIN965" (at 222.25 85.09 0)
+      (effects (font (size 1.27 1.27)) hide)
+    )
+    (property "Datasheet" "~" (at 222.25 85.09 0)
+      (effects (font (size 1.27 1.27)) hide)
+    )
+    (instances
+      (project "DDRN_Hardware"
+        (path "/6ac82b7e-9b2f-410f-b4a2-ac71ebf885a9"
+          (reference "H4") (unit 1)
+        )
+      )
+    )
+  )
   (symbol (lib_id "Connector:Conn_01x02_Pin") (at 116.84 29.21 0) (unit 1)
     (in_bom yes) (on_board yes) (dnp no) (fields_autoplaced)
@@
         (path "/6ac82b7e-9b2f-410f-b4a2-ac71ebf885a9"
           (reference "#PWR01") (unit 1)
+        )
+      )
+    )
+  )
+  (symbol (lib_id "Mechanical:MountingHole") (at 222.25 69.85 0) (unit 1)
+    (in_bom yes) (on_board yes) (dnp no) (fields_autoplaced)
+    (property "Reference" "H1" (at 224.79 68.58 0)
+      (effects (font (size 1.27 1.27)) (justify left))
+    )
+    (property "Value" "MountingHole" (at 224.79 71.12 0)
+      (effects (font (size 1.27 1.27)) (justify left))
+    )
+    (property "Footprint" "MountingHole:MountingHole_3.2mm_M3_DIN965" (at 222.25 69.85 0)
+      (effects (font (size 1.27 1.27)) hide)
+    )
+    (property "Datasheet" "~" (at 222.25 69.85 0)
+      (effects (font (size 1.27 1.27)) hide)
+    )
+    (instances
+      (project "DDRN_Hardware"
+        (path "/6ac82b7e-9b2f-410f-b4a2-ac71ebf885a9"
+          (reference "H1") (unit 1)
         )
       )
@@
       (effects (font (size 1.27 1.27)))
     )
-    (property "Footprint" "Library:bmp390_handsolder" (at 53.34 163.83 0)
+    (property "Footprint" "Library:lsm303_handsolder" (at 53.34 163.83 0)
       (effects (font (size 1.27 1.27)) (justify bottom) hide)
     )

Commit message: moving files
Parts:
- added J1: Conn_01x03_Pin, Connector_PinHeader_2.54mm:PinHeader_1x03_P2.54mm_Vertical, symbol Connector:Conn_01x03_Pin
- added J6, J7, J9: Conn_01x02_Pin, Connector_PinHeader_2.54mm:PinHeader_1x02_P2.54mm_Vertical, symbol Connector:Conn_01x02_Pin
- added R19: 1k, Resistor_SMD:R_0805_2012Metric_Pad1.20x1.40mm_HandSolder, symbol Device:R_Small_US
- added SW2: SW_Push, Button_Switch_SMD:SW_SPST_PTS810, symbol Switch:SW_Push
Connections:
- net 3v3: now also J9.2 (Pin_2), R19.2
- net Anneal_Enable: now also J7.2 (Pin_2)
- net Battery_Monitor: now also J1.3 (Pin_3)
- net GND: now also J6.1 (Pin_1), J9.1 (Pin_1), SW2.2
- net SiPM_Bias: now also J6.2 (Pin_2)
- net SiPM_Signal: now also J1.2 (Pin_2)
- net SiPM_Temp: now also J1.1 (Pin_1)
- net Stim_Enable: now also J7.1 (Pin_1)
- net Boot_Mode: now reaches U1.18 (PA3)
- net Boot_Mode: now also R19.1, SW2.1
Other:
- moved on the sheet: C10, C7, C8, C9, R14, SW1, U6
