File: LED_Study/pcb/LED_board_XEG/LED_board.kicad_sch (KiCad schematic)
At the start: 4 parts

Commit message: updated boards and ordered from PCBway
Parts:
- added J1, J2: Conn_01x01_Pin, Connector_PinHeader_1.00mm:PinHeader_1x01_P1.00mm_Vertical, symbol Connector:Conn_01x01_Pin
Connections:
- net GND: now also J2.1 (Pin_1)
- net Vin: now also J1.1 (Pin_1)
Changed lines of the file:
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@@
+    )
+  )
+  (symbol (lib_id "Connector:Conn_01x01_Pin") (at 69.85 39.37 0) (unit 1)
+    (in_bom yes) (on_board yes) (dnp no) (fields_autoplaced)
+    (property "Reference" "J1" (at 70.485 34.29 0)
+      (effects (font (size 1.27 1.27)))
+    )
+    (property "Value" "Conn_01x01_Pin" (at 70.485 36.83 0)
+      (effects (font (size 1.27 1.27)))
+    )
+    (property "Footprint" "Connector_PinHeader_1.00mm:PinHeader_1x01_P1.00mm_Vertical" (at 69.85 39.37 0)
+      (effects (font (size 1.27 1.27)) hide)
+    )
+    (property "Datasheet" "~" (at 69.85 39.37 0)
+      (effects (font (size 1.27 1.27)) hide)
+    )
+    (pin "1")
+    (instances
+      (project "LED_board"
+        (path "/ee3210f4-4163-4542-8403-a0d7023a83cd"
+          (reference "J1") (unit 1)
+        )
+      )
     )
   )
@@
         )
       )
+    )
+  )
+  (symbol (lib_id "Connector:Conn_01x01_Pin") (at 63.5 72.39 0) (unit 1)
+    (in_bom yes) (on_board yes) (dnp no) (fields_autoplaced)
+    (property "Reference" "J2" (at 64.135 67.31 0)
+      (effects (font (size 1.27 1.27)))
+    )
+    (property "Value" "Conn_01x01_Pin" (at 64.135 69.85 0)
+      (effects (font (size 1.27 1.27)))
+    )
+    (property "Footprint" "Connector_PinHeader_1.00mm:PinHeader_1x01_P1.00mm_Vertical" (at 63.5 72.39 0)
+      (effects (font (size 1.27 1.27)) hide)
+    )
+    (property "Datasheet" "~" (at 63.5 72.39 0)
+      (effects (font (size 1.27 1.27)) hide)
+    )
+    (pin "1")
+    (instances
+      (project "LED_board"
+        (path "/ee3210f4-4163-4542-8403-a0d7023a83cd"
+          (reference "J2") (unit 1)
+        )
+      )
